File: XY_RJ12_breakout.sch (EAGLE design)
At the start: 36 parts

Commit message: Fix wrong label on XSTEPPER and YSTEPPER port
Parts:
- renumbered XSERVO to XSTEPPER, YSERVO to YSTEPPER
Changed lines of the file:
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@@
 <parts>
 <part name="XLIMIT" library="con-rj" deviceset="RJ12" device=""/>
-<part name="XSERVO" library="con-rj" deviceset="RJ12" device=""/>
-<part name="YSERVO" library="con-rj" deviceset="RJ12" device=""/>
+<part name="XSTEPPER" library="con-rj" deviceset="RJ12" device=""/>
+<part name="YSTEPPER" library="con-rj" deviceset="RJ12" device=""/>
 <part name="YLIMIT" library="con-rj" deviceset="RJ12" device=""/>
 <part name="SERVO" library="con-rj" deviceset="RJ12" device=""/>
@@
 <instances>
 <instance part="XLIMIT" gate="G$1" x="15.24" y="55.88"/>
-<instance part="XSERVO" gate="G$1" x="15.24" y="-2.54"/>
-<instance part="YSERVO" gate="G$1" x="15.24" y="25.4"/>
+<instance part="XSTEPPER" gate="G$1" x="15.24" y="-2.54"/>
+<instance part="YSTEPPER" gate="G$1" x="15.24" y="25.4"/>
 <instance part="YLIMIT" gate="G$1" x="15.24" y="86.36"/>
 <instance part="SERVO" gate="G$1" x="15.24" y="116.84"/>
@@
 <junction x="-149.86" y="78.74"/>
 <pinref part="JP1" gate="G$1" pin="1"/>
-<pinref part="YSERVO" gate="G$1" pin="3"/>
+<pinref part="YSTEPPER" gate="G$1" pin="3"/>
 <wire x1="-99.06" y1="22.86" x2="5.08" y2="22.86" width="0.1524" layer="91"/>
-<pinref part="XSERVO" gate="G$1" pin="3"/>
+<pinref part="XSTEPPER" gate="G$1" pin="3"/>
 <wire x1="-101.6" y1="-5.08" x2="5.08" y2="-5.08" width="0.1524" layer="91"/>
 </segment>
@@
 <junction x="-149.86" y="73.66"/>
 <pinref part="JP3" gate="G$1" pin="1"/>
-<pinref part="XSERVO" gate="G$1" pin="4"/>
+<pinref part="XSTEPPER" gate="G$1" pin="4"/>
 <wire x1="-83.82" y1="-2.54" x2="5.08" y2="-2.54" width="0.1524" layer="91"/>
-<pinref part="YSERVO" gate="G$1" pin="4"/>
+<pinref part="YSTEPPER" gate="G$1" pin="4"/>
 <wire x1="5.08" y1="25.4" x2="-83.82" y2="25.4" width="0.1524" layer="91"/>
 <junction x="-83.82" y="25.4"/>
@@
 <wire x1="-142.24" y1="55.88" x2="-104.14" y2="55.88" width="0.1524" layer="91"/>
 <wire x1="-104.14" y1="55.88" x2="-104.14" y2="20.32" width="0.1524" layer="91"/>
-<pinref part="YSERVO" gate="G$1" pin="2"/>
+<pinref part="YSTEPPER" gate="G$1" pin="2"/>
 <wire x1="-104.14" y1="20.32" x2="5.08" y2="20.32" width="0.1524" layer="91"/>
 <pinref part="JP10" gate="G$1" pin="1"/>
@@
 <wire x1="-142.24" y1="53.34" x2="-106.68" y2="53.34" width="0.1524" layer="91"/>
 <wire x1="-106.68" y1="53.34" x2="-106.68" y2="17.78" width="0.1524" layer="91"/>
-<pinref part="YSERVO" gate="G$1" pin="1"/>
+<pinref part="YSTEPPER" gate="G$1" pin="1"/>
 <wire x1="-106.68" y1="17.78" x2="5.08" y2="17.78" width="0.1524" layer="91"/>
 <pinref part="JP11" gate="G$1" pin="1"/>
@@
 <wire x1="-142.24" y1="50.8" x2="-109.22" y2="50.8" width="0.1524" layer="91"/>
 <wire x1="-109.22" y1="50.8" x2="-109.22" y2="-7.62" width="0.1524" layer="91"/>
-<pinref part="XSERVO" gate="G$1" pin="2"/>
+<pinref part="XSTEPPER" gate="G$1" pin="2"/>
 <wire x1="-109.22" y1="-7.62" x2="5.08" y2="-7.62" width="0.1524" layer="91"/>
 <pinref part="JP12" gate="G$1" pin="1"/>
@@
 <wire x1="-142.24" y1="48.26" x2="-111.76" y2="48.26" width="0.1524" layer="91"/>
 <wire x1="-111.76" y1="48.26" x2="-111.76" y2="-10.16" width="0.1524" layer="91"/>
-<pinref part="XSERVO" gate="G$1" pin="1"/>
+<pinref part="XSTEPPER" gate="G$1" pin="1"/>
 <wire x1="-111.76" y1="-10.16" x2="5.08" y2="-10.16" width="0.1524" layer="91"/>
 <pinref part="JP13" gate="G$1" pin="1"/>
